File: pcb/face/face.kicad_pcb (KiCad board)
At the start: 2 copper layers, 101.5 x 52 mm, 29 parts, among them J1 Screw_Terminal_01x02, J2 Screw_Terminal_01x05, J3 Screw_Terminal_01x05, J4 282856-2, Q1 IRLB8721PBF, Q2 IRLB8721PBF, Q5 IRLB8721PBF, Q6 IRLB8721PBF, U1 SN65HVD230DR, U2 PicoW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

Commit message: Final boards
Parts:
- removed U4: NCP1117-3.3_SOT223, Package_TO_SOT_SMD:SOT-223-3_TabPin2
- added U6: NCP1117-5.0_SOT223, Package_TO_SOT_SMD:SOT-223-3_TabPin2, F.Cu at (90.8, 66.0)
- R5, R6: value 60Ω -> 240Ω; footprint Resistor_SMD:R_1206_3216Metric -> Resistor_SMD:R_0603_1608Metric
Connections:
- C2 pad 1: VSYS -> +3V3
- C3 pad 1: VSYS -> +3V3
- R3 pad 1: VSYS -> +3V3
- U1 pad 3: VSYS -> +3V3
- U2 pad 36: unconnected-(U2-3V3-Pad36)_1 -> +3V3
- U3 pad 2: VSYS -> +3V3
Routing:
- net +3V3: track 0.00 -> 73.2 mm
- net VSYS: track 77.9 -> 8.14 mm
- net Net-(D2-K): track 3.04 -> 3.67 mm
- net Net-(D1-K): track 3.04 -> 3.67 mm
- net GND: track 26.7 -> 27.3 mm
- added copper zone on F.Cu, net +3V3
- removed copper zone on F.Cu, net VSYS
Other:
- board text added: "+12V"
- board text added: "12V Input"
- board text added: "Blue"
- board text added: "CANH"
- board text added: "CANL"
- board text added: "GND"
- board text added: "Green"
- board text added: "McGraw Tower LED Driver"
- board text added: "Red"
- board text added: "White"
