File: pcb/face/face.kicad_sch (KiCad schematic)
At the start: 15 parts, among them Q1 IRLB8721PBF, Q2 IRLB8721PBF, Q5 IRLB8721PBF, Q6 IRLB8721PBF, U1 SN65HVD230DR, U2 PicoW, U3 FDN340P

Commit message: PCBs hopefully done
Parts:
- added C4, C5: 10μF, Capacitor_SMD:C_0603_1608Metric, symbol Device:C
- added D1, D2: LED, LED_THT:LED_D5.0mm, symbol Device:LED
- added H1, H2: MountingHole, MountingHole:MountingHole_3.2mm_M3_DIN965_Pad, symbol Mechanical:MountingHole
- added J1: Screw_Terminal_01x02, TerminalBlock_Phoenix:TerminalBlock_Phoenix_PT-1,5-2-5.0-H_1x02_P5.00mm_Horizontal, symbol Connector:Screw_Terminal_01x02
- added J2, J3: Screw_Terminal_01x05, TerminalBlock_Phoenix:TerminalBlock_Phoenix_PT-1,5-5-5.0-H_1x05_P5.00mm_Horizontal, symbol Connector:Screw_Terminal_01x05
- added J4: 282856-2, 282856-2:TE_282856-2, symbol 282856-2:282856-2
- added R5, R6: 60Ω, Resistor_SMD:R_1206_3216Metric, symbol Device:R
- added U4: NCP1117-3.3_SOT223, Package_TO_SOT_SMD:SOT-223-3_TabPin2, symbol Regulator_Linear:NCP1117-3.3_SOT223
- added U5: DMG2305UX-7, dmg2305ux:SOT-23_DIO, symbol dmg2305ux:DMG2305UX-7
- U1: footprint CAN:D8 -> can:D8
Connections:
- net CANH: now also J1.1 (Pin_1)
- net CANL: now also J1.2 (Pin_2)
- net GATE_B: now also U2.26 (GPIO20); no longer U2.25 (GPIO19)
- net GATE_G: now also U2.31 (GPIO26_ADC0); no longer U2.26 (GPIO20)
- net GATE_R: now also U2.34 (GPIO28_ADC2); no longer U2.27 (GPIO21)
- net GND: now also C4.2, C5.2, J4.2, R5.2, R6.2, U4.1 (GND)
- net LED_B: now also J2.4 (Pin_4), J3.2 (Pin_2)
- net LED_G: now also J2.3 (Pin_3), J3.3 (Pin_3)
- net LED_R: now also J2.2 (Pin_2), J3.4 (Pin_4)
- net LED_W: now also J2.5 (Pin_5), J3.1 (Pin_1)
- net VBUS: now also U5.1
- net VSYS: now also U5.2
- new net: D2.1 (K), R6.1
- new net: D1.1 (K), R5.1
- new net +12V: C4.1, J2.1 (Pin_1), J3.5 (Pin_5), J4.1, U4.3 (VI)
- new net LED_COMM: D2.2 (A), U2.25 (GPIO19)
- new net LED_ON: D1.2 (A), U2.27 (GPIO21)
- new net VCONV: C5.1, U4.2 (VO), U5.3
- no-connect marks 25 -> 23
Other:
- note added: "CAN Outputs"
- note added: "Mounting"
- note added: "Power"
- note added: "Status LEDs"
- title: (none) -> McGraw Tower LED Driver

Commit message: Final boards
Parts:
- removed U4: NCP1117-3.3_SOT223, Package_TO_SOT_SMD:SOT-223-3_TabPin2, symbol Regulator_Linear:NCP1117-3.3_SOT223
- added U6: NCP1117-5.0_SOT223, Package_TO_SOT_SMD:SOT-223-3_TabPin2, symbol Regulator_Linear:NCP1117-5.0_SOT223
- R5, R6: value 60Ω -> 240Ω; footprint Resistor_SMD:R_1206_3216Metric -> Resistor_SMD:R_0603_1608Metric
Connections:
- net +12V: now also U6.3 (VI)
- net GND: now also U6.1 (GND)
- net VCONV: now also U6.2 (VO)
- net VSYS: no longer C2.1, C3.1, R3.1, U1.3 (VCC), U3.2
- net +3V3: now reaches U2.36 (3V3)
- net +3V3: now also C2.1, C3.1, R3.1, U1.3 (VCC), U3.2
- no-connect marks 23 -> 22
