File: pcb/sensor/sensor.kicad_pcb (KiCad board)
At the start: 2 copper layers, 52 x 65 mm, 21 parts, among them J1 PPTC031LFBN-RC, J2 Barrel_Jack_MountingPin, J3 Screw_Terminal_01x02, U1 SN65HVD230DR, U2 FDN340P, U3 PicoW, U4 VEML6030-GS15, U5 DMG2305UX-7

Commit message: Final boards
Connections:
- C2 pad 1: VSYS -> +3V3
- C3 pad 1: VSYS -> +3V3
- J1 pad 3: VSYS -> +3V3
- R3 pad 1: VSYS -> +3V3
- R5 pad 1: VSYS -> +3V3
- R6 pad 1: VSYS -> +3V3
- R7 pad 1: VSYS -> +3V3
- U1 pad 3: VSYS -> +3V3
- U2 pad 2: VSYS -> +3V3
- U3 pad 36: unconnected-(U3-3V3-Pad36) -> +3V3
- U4 pad 4: VSYS -> +3V3
- U4 pad 6: VSYS -> +3V3
Routing:
- net +3V3: track 0.00 -> 58.1 mm
- net VSYS: track 70.5 -> 16.3 mm
- added copper zone on F.Cu, net +3V3
- removed copper zone on F.Cu, net VSYS
Other:
- board text added: "McGraw Tower LED Sensor Board"
- board text removed: "LED Sensor Board"
