File: pcb/sensor/sensor.kicad_sch (KiCad schematic)
At the start: 11 parts, among them U1 SN65HVD230DR, U2 FDN340P, U3 PicoW

Commit message: Worked on PCBs
Parts:
- added R5, R6: 4.7KΩ, symbol Device:R
- added R7: 10KΩ, symbol Device:R
- added U4: VEML6030-GS15, veml6030_gs15:VISHAY_VEML6030_2X2X0.87, symbol veml6030_gs15:VEML6030-GS15
Connections:
- net GND: now also U4.1
- net VSYS: now also R5.1, R6.1, R7.1, U4.4, U4.6
- net L_INT: now reaches U3.25 (GPIO19)
- net L_INT: now also R7.2, U4.3
- net L_SDA: now reaches U3.26 (GPIO20)
- net L_SDA: now also R5.2, U4.2
- net L_SCL: now reaches U3.27 (GPIO21)
- net L_SCL: now also R6.2, U4.5
- no-connect marks 29 -> 26
Other:
- note added: "Default Addr: 0x48"
- note added: "Light Sensor"

Commit message: Incremental PCB
Parts:
- added J1: PPTC031LFBN-RC, CONN_PPTC031_SUL, symbol pptc031lfbn:PPTC031LFBN-RC
Connections:
- net GND: now also J1.2
- net VSYS: now also J1.3
- new net MIC: J1.1
Other:
- note added: "Microphone"

Commit message: PCBs hopefully done
Parts:
- added H1, H2: MountingHole, MountingHole:MountingHole_3.2mm_M3_DIN965_Pad, symbol Mechanical:MountingHole
- added J2: Barrel_Jack_MountingPin, Connector_BarrelJack:BarrelJack_CUI_PJ-102AH_Horizontal, symbol Connector:Barrel_Jack_MountingPin
- added J3: Screw_Terminal_01x02, TerminalBlock_Phoenix:TerminalBlock_Phoenix_PT-1,5-2-5.0-H_1x02_P5.00mm_Horizontal, symbol Connector:Screw_Terminal_01x02
- added U5: DMG2305UX-7, dmg2305ux:SOT-23_DIO, symbol dmg2305ux:DMG2305UX-7
- J1: footprint CONN_PPTC031_SUL -> pptc031lfbn:CONN_PPTC031_SUL
- R5, R6, R7: footprint (none) -> Resistor_SMD:R_0603_1608Metric
Connections:
- net CANH: now also J3.1 (Pin_1)
- net CANL: now also J3.2 (Pin_2)
- net GND: now also J2.2
- net MIC: now also U3.31 (GPIO26_ADC0)
- net VBUS: now also U5.1
- net VSYS: now also U5.2
- new net VBARREL: J2.1, U5.3
Other:
- note added: "5V Supply"
- note added: "CAN Outputs"
- note added: "Mounting"
- note added: "Power"

Commit message: Final boards
Connections:
- net VSYS: no longer C2.1, C3.1, J1.3, R3.1, R5.1, R6.1, R7.1, U1.3 (VCC), U2.2, U4.4, U4.6
- net +3V3: now reaches U3.36 (3V3)
- net +3V3: now also C2.1, C3.1, J1.3, R3.1, R5.1, R6.1, R7.1, U1.3 (VCC), U2.2, U4.4, U4.6
- no-connect marks 26 -> 25
